Commit message: Add IMU and publish TF frames
It is crucial that every link has inertia (check `imu_link`), otherwise Gazebo will not create it and its parent joint.

File: urdf/dummy.urdf (robot description, URDF)
Before this commit: robot dummy, 2 links, 1 joints
Links:
- added link imu_link, mass 0.01
Joints:
- added joint imu_joint: type revolute, parent base_link, child imu_link, origin xyz=0 0 0 rpy=0 0 0, axis 0 0 1, limit lower=0 upper=0 effort=0 velocity=0

Commit message: Add forward-looking and mechanical sonars
Sonar courtesy of Brazilian Institute of Robotics

File: urdf/dummy.urdf (robot description, URDF)
Before this commit: robot dummy, 3 links, 2 joints
Links:
- removed link sonar_link
- added link mbe_sonar_link, mass 0.78; collision box size=0.1 0.1 0.1; visual box size=0.11 0.1 0.0423
- added link ping360_sonar_link, mass 0.01; collision box size=0.1 0.1 0.1; visual cylinder length=0.12 radius=0.04
Joints:
- removed joint sonar_joint
- added joint mbe_sonar_joint: type revolute, parent base_link, child mbe_sonar_link, origin xyz=0.15 0 -0.2 rpy=0 0.174533 0, axis 0 0 1, limit lower=0 upper=0 effort=0 velocity=0
- added joint ping360_sonar_joint: type revolute, parent base_link, child ping360_sonar_link, origin xyz=0.15 0 0.175 rpy=0 0 0, axis 0 0 1, limit lower=0 upper=0 effort=0 velocity=0
