Commit message: Add Ping2 altimeter

File: model/sonars.urdf.xacro (robot description, xacro)
@@ -3,5 +3,5 @@
 	<xacro:property name="deg2rad" value="${pi / 180}"/>
 	<!-- ================================= -->
-	<!-- Macro for the sonar sensor itself -->
+	<!-- Macro for sonar sensor -->
 	<xacro:macro name="sonar_macro" params=
 		"sonar_link topic hfov vfov bin_count beam_count image_width image_height
@@ -72,4 +72,45 @@
 		</gazebo>
 	</xacro:macro>
+	<!-- =================== -->
+	<!-- Macro for altimeter -->
+	<xacro:macro name="altimeter_macro" params=
+		"alti_link topic update_rate range_min range_max range_resolution
+		noise_mean noise_stddev visualize:=true prefix:=^ namespace:=^ gravity:=^"
+	>
+		<gazebo reference="${alti_link}">
+			<!-- Plugin for altimeter -->
+			<xacro:unless value="${gravity}">
+				<turnGravityOff>1</turnGravityOff>
+			</xacro:unless>
+			<sensor type="ray" name="Altimeter">
+				<visualize>${visualize}</visualize>
+				<update_rate>${update_rate}</update_rate>
+				<ray>
+					<scan>
+						<horizontal>
+						<samples>1</samples>
+						<resolution>1</resolution>
+						<min_angle>0.0</min_angle>
+						<max_angle>0.0</max_angle>
+						</horizontal>
+					</scan>
+					<range>
+						<min>${range_min}</min>
+						<max>${range_max}</max>
+						<resolution>${range_resolution}</resolution>
+					</range>
+					<noise>
+						<type>gaussian</type>
+						<mean>${noise_mean}</mean>
+						<stddev>${noise_stddev}</stddev>
+					</noise>
+				</ray>
+				<plugin name="Altimeter" filename="libgazebo_ros_laser.so">
+					<topicName>${namespace}/${topic}</topicName>
+					<frameName>${alti_link}</frameName>
+				</plugin>
+			</sensor>
+		</gazebo>
+	</xacro:macro>
 	<!-- ================= -->
 	<!-- Macro for Ping360 -->
@@ -160,3 +201,40 @@
 		/>
 	</xacro:macro>
+	<!-- ================= -->
+	<!-- Macro for Ping2 -->
+	<xacro:macro name="ping2_macro" params="parent_link *joint_origin *joint_axis prefix:='' namespace:='' gravity:=true">
+		<link name="${prefix}ping2_link">
+			<inertial>
+				<mass value="0.01" />
+				<origin xyz="0 0 0" rpy="0 0 0" />
+				<inertia ixx="0.01" ixy="0.001" ixz="0.001" iyy="0.01" iyz="0.001" izz="0.01" />
+			</inertial>
+			<visual name="visual">
+				<origin xyz="0 0 0" rpy="0 1.57079632679 0" />
+				<geometry>
+					<cylinder length="0.041" radius="0.025" />
+				</geometry>
+			</visual>
+			<collision>
+				<origin xyz="0 0 0" rpy="0 0 0" />
+				<geometry>
+					<box size="0.1 0.1 0.1" />
+				</geometry>
+			</collision>
+		</link>
+		<joint name="${prefix}ping2_joint" type="revolute">
+			<xacro:insert_block name="joint_origin"/>
+			<xacro:insert_block name="joint_axis"/>
+			<parent link="${parent_link}" />
+			<child link="${prefix}ping2_link" />
+			<limit upper="0" lower="0" effort="0" velocity="0" />
+		</joint>
+		<!-- Add the altimeter plugin -->
+		<xacro:altimeter_macro
+			alti_link="${prefix}ping2_link" topic="ping2_ray"
+			update_rate="5" range_min="0.3" range_max="50" range_resolution="0.01"
+			noise_mean="0.0" noise_stddev="0.05" visualize="true"
+			prefix="${prefix}" namespace="${namespace}" gravity="${gravity}"
+		/>
+	</xacro:macro>
 </robot>

File: robots/dummy.urdf.xacro (robot description, xacro)
@@ -86,5 +86,5 @@
 			<robotNamespace>dummy</robotNamespace>
 			<!-- Must have this list of joints -->
-			<jointName>imu_joint, ping360_sonar_joint, mbe_sonar_joint</jointName>
+			<jointName>imu_joint, ping360_sonar_joint, mbe_sonar_joint, ping2_joint</jointName>
 			<updateRate>30</updateRate>
 		</plugin>
@@ -100,4 +100,5 @@
 	</gazebo>
 	<!-- Mount the sonars -->
+  <!-- Attention: need to update joint_state_publisher above-->
 	<xacro:include filename="../model/sonars.urdf.xacro"/>
 	<xacro:ping360_macro parent_link="base_link" namespace="/dummy" gravity="false">
@@ -109,3 +110,7 @@
     <axis xyz="0 0 1"/>
 	</xacro:mbe_macro>
+	<xacro:ping2_macro parent_link="base_link" namespace="/dummy" gravity="false">
+    <origin xyz="0.0 0.15 -0.175" rpy="0 1.57079632679 0" />
+    <axis xyz="0 0 1" />
+	</xacro:ping2_macro>
 </robot>

File: urdf/dummy.urdf (robot description, URDF)
Before this commit: robot dummy, 4 links, 3 joints
Links:
- added link ping2_link, mass 0.187; collision box size=0.1 0.1 0.1; visual cylinder length=0.041 radius=0.025
Joints:
- added joint ping2_joint: type revolute, parent base_link, child ping2_link, origin xyz=0.0 0.15 -0.175 rpy=0 1.57079632679 0, axis 0 0 1, limit lower=0 upper=0 effort=0 velocity=0

Commit message: Update Ping360 dimensions

File: model/sonars.urdf.xacro (robot description, xacro)
@@ -124,5 +124,5 @@
 				<origin xyz="0 0 0" rpy="0 0 0" />
 				<geometry>
-					<cylinder length="0.12" radius="0.04" />
+					<cylinder length="0.083" radius="0.0385" />
 				</geometry>
 			</visual>
