Commit message: Fix faux depth camera orientation

File: models/sonars.urdf.xacro (robot description, xacro)
@@ -7,5 +7,5 @@
 		"sonar_link topic hfov vfov bin_count beam_count image_width image_height
 		clip_near clip_far image_format=R32G32B32 disable_color:=true
-		faux_depth:=false faux_depth_namespace:=''
+		faux_depth:=false faux_depth_link:='' faux_depth_namespace:=''
 		prefix:=^ namespace:=^ gravity:=^"
 	>
@@ -63,5 +63,5 @@
 						<depthImageCameraInfoTopicName>${namespace}/${faux_depth_namespace}/depth/camera_info</depthImageCameraInfoTopicName>
 						<pointCloudTopicName>${namespace}/${faux_depth_namespace}/depth/points</pointCloudTopicName>
-						<frameName>${sonar_link}</frameName>
+						<frameName>${faux_depth_link}</frameName>
 						<pointCloudCutoff>${clip_near}</pointCloudCutoff>
 						<pointCloudCutoffMax>${clip_far}</pointCloudCutoffMax>
@@ -141,10 +141,24 @@
 			<limit upper="0" lower="0" effort="0" velocity="0" />
 		</joint>
+		<link name="${prefix}ping360_depth_link">
+			<inertial>
+				<mass value="0.0001" />
+				<origin xyz="0 0 0" rpy="0 0 0" />
+				<inertia ixx="0.0001" ixy="0.0001" ixz="0.0001" iyy="0.0001" iyz="0.0001" izz="0.0001" />
+			</inertial>
+		</link>
+		<joint name="${prefix}ping360_depth_joint" type="revolute">
+			<origin xyz="0 0 0" rpy="-1.57079632679 0 -1.57079632679"/>
+			<axis xyz="0 0 1"/>
+			<parent link="${prefix}ping360_sonar_link" />
+			<child link="${prefix}ping360_depth_link" />
+			<limit upper="0" lower="0" effort="0" velocity="0" />
+		</joint>
 		<!-- Add the sonar plugin -->
 		<xacro:sonar_macro
 			sonar_link="${prefix}ping360_sonar_link" topic="ping360_sonar"
 			hfov="${120*deg2rad}" vfov="${25*deg2rad}" bin_count="1024" beam_count="128"
-			image_width="1024" image_height="1024" clip_near="0.75" clip_far="10.0"
-			image_format="R8G8B8" faux_depth="true" faux_depth_namespace="ping360_sim_depth"
+			image_width="1024" image_height="1024" clip_near="0.75" clip_far="10.0" image_format="R8G8B8"
+			faux_depth="true" faux_depth_link="${prefix}ping360_depth_link" faux_depth_namespace="ping360_sim_depth"
 			prefix="${prefix}" namespace="${namespace}" gravity="${gravity}"
 		/>

File: robots/dummy.urdf.xacro (robot description, xacro)
@@ -86,5 +86,5 @@
 			<robotNamespace>dummy</robotNamespace>
 			<!-- Must have this list of joints -->
-			<jointName>imu_joint, ping360_sonar_joint, mbe_sonar_joint, ping2_joint</jointName>
+			<jointName>imu_joint, ping360_sonar_joint, mbe_sonar_joint, ping2_joint, ping360_depth_joint</jointName>
 			<updateRate>30</updateRate>
 		</plugin>
@@ -101,5 +101,5 @@
 	<!-- Mount the sonars -->
   <!-- Attention: need to update joint_state_publisher above-->
-	<xacro:include filename="../model/sonars.urdf.xacro"/>
+	<xacro:include filename="../models/sonars.urdf.xacro"/>
 	<xacro:ping360_macro parent_link="base_link" namespace="/dummy" gravity="false">
 		<origin xyz="0.15 0 0.175" rpy="0 0 0"/>

Commit message: CHG make mass negligable to avoid shifting center of mass

File: models/sonars.urdf.xacro (robot description, xacro)
@@ -117,5 +117,5 @@
 		<link name="${prefix}ping360_sonar_link">
 			<inertial>
-				<mass value="0.1" />
+				<mass value="0.00001" />
 				<origin xyz="0 0 0" rpy="0 0 0" />
 				<inertia ixx="0.01" ixy="0.001" ixz="0.001" iyy="0.01" iyz="0.001" izz="0.01" />
@@ -169,5 +169,6 @@
 		<link name="${prefix}mbe_sonar_link">
 			<inertial>
-				<mass value="0.78" />
+				<!-- <mass value="0.78" /> -->
+				<mass value="0.00001" />
 				<origin xyz="0 0 0" rpy="0 0 0" />
 				<inertia ixx="0.01" ixy="0.001" ixz="0.001" iyy="0.01" iyz="0.001" izz="0.01" />
@@ -219,5 +220,5 @@
 		<link name="${prefix}ping2_link">
 			<inertial>
-				<mass value="0.01" />
+				<mass value="0.00001" />
 				<origin xyz="0 0 0" rpy="0 0 0" />
 				<inertia ixx="0.01" ixy="0.001" ixz="0.001" iyy="0.01" iyz="0.001" izz="0.01" />
